File: hardware/pcb/meaco-attiny.kicad_pcb (KiCad board)
At the start: 2 copper layers, 35.1 x 32 mm, 17 parts, among them J1 Conn_02x03_Odd_Even, J2 Conn_01x04_Male, J3 Conn_01x02_Male, J4 Conn_01x02_Male, Q1 2N3904, SW1 SW_Push, U1 ATtiny85-20P

Commit message: JLC! JLC! JLC! JLC!
Other:
- board text added: "JLCJLCJLCJLC"
Changed lines of the file:
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@@
   (gr_arc (start 114.538741 157.249809) (mid 103.281511 153.877371) (end 95.514261 145.058732) (layer "B.SilkS") (width 0.5))
   (gr_arc (start 108.778762 140.11476) (mid 107.938537 133.239537) (end 113.176419 128.707512) (layer "B.SilkS") (width 0.5))
-  (gr_arc (start 106.439024 138.050271) (mid 106.241866 134.720855) (end 107.320067 131.564693) (layer "B.SilkS") (width 0.5))
+  (gr_arc (start 106.439024 138.050271) (mid 106.241866 134.720856) (end 107.320067 131.564693) (layer "B.SilkS") (width 0.5))
   (gr_arc (start 123.785605 140.077568) (mid 116.02289 145.722094) (end 107.119317 142.13785) (layer "B.SilkS") (width 0.5))
-  (gr_arc (start 110.490515 128.412257) (mid 121.683033 130.660484) (end 120.86527 142.047242) (layer "B.SilkS") (width 0.5))
+  (gr_arc (start 110.490515 128.412257) (mid 121.683034 130.660484) (end 120.86527 142.047242) (layer "B.SilkS") (width 0.5))
   (gr_arc (start 116.385666 130.001205) (mid 120.65631 137.613646) (end 112.938241 141.690293) (layer "B.SilkS") (width 0.5))
   (gr_arc (start 102.532035 144.485129) (mid 103.09622 126.540303) (end 120.470234 122.014963) (layer "B.SilkS") (width 0.5))
   (gr_arc (start 117.876066 119.924224) (mid 121.672246 121.151982) (end 125.054954 123.267556) (layer "B.SilkS") (width 0.5))
-  (gr_arc (start 96.008401 135.637986) (mid 102.087992 122.047885) (end 116.143716 117.139838) (layer "B.SilkS") (width 0.5))
+  (gr_arc (start 96.008401 135.637986) (mid 102.087992 122.047884) (end 116.143716 117.139838) (layer "B.SilkS") (width 0.5))
   (gr_circle (center 114.808 135.89) (end 118.418018 135.89) (layer "B.SilkS") (width 0.15) (fill solid))
   (gr_arc (start 134.777073 137.906217) (mid 129.534302 149.535837) (end 118.34301 155.658722) (layer "B.SilkS") (width 0.5))
@@
     (effects (font (size 0.8 0.8) (thickness 0.15)))
   )
+  (gr_text "JLCJLCJLCJLC" (at 111.76 137.16) (layer "F.SilkS")
+    (effects (font (size 0.8 0.8) (thickness 0.15)))
+  )
